File: ESC_Texas/ESC_Texas.kicad_sch (KiCad schematic)
At the start: 83 parts, among them IC1 nRF52840-QFAA-F-R7, IC11 LM3480IM3-3.3_NOPB, IC12 LM3480IM3-3.3_NOPB, IC16 MC78L05ACHT1G, J11 input-10V, J12 Hall Effect, J13 Conn_01x04_Pin, J14 Conn_01x01_Pin, J17 Conn_01x01_Pin, J2 BD125-10-A-0305-0580-L-B, J3 Motor, J4 Conn_01x02_Pin, P0.03 TestPoint, P0.08 TestPoint, P0.09 TestPoint, P0.10 TestPoint, P0.11 TestPoint, P0.12 TestPoint, P0.7 TestPoint, P1.0 TestPoint, P1.9 TestPoint, U1 MCP2515-xSO, U2 TJA1051T, X1 CM7V-T1A-32.768kHz, X2 32MHz, X3 C115962

Commit message: filters
Parts:
- added C19: F, Capacitor_SMD:C_0805_2012Metric, symbol Device:C
- added R31: R, Resistor_SMD:R_0805_2012Metric, symbol Device:R
- renumbered P0.7 to P0.07, P1.9 to P1.09
Connections:
- net GND: now also C19.2
- net P0.04: now also C19.1, R31.1
- new net Battery-Current/Current-Sense: R31.2
Changed lines of the file:
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@@
 	)
 	(junction
+		(at 201.93 68.58)
+		(diameter 0)
+		(color 0 0 0 0)
+	)
+	(junction
 		(at 72.39 175.26)
 		(diameter 0)
@@
 	(wire
 		(pts
+			(xy 201.93 68.58) (xy 201.93 71.12)
+		)
+		(stroke
+			(width 0)
+			(type default)
+		)
+	)
+	(wire
+		(pts
 			(xy 86.36 257.81) (xy 86.36 260.35)
 		)
@@
 	(wire
 		(pts
-			(xy 193.04 68.58) (xy 200.66 68.58)
-		)
-		(stroke
-			(width 0)
-			(type default)
-		)
-	)
-	(wire
-		(pts
 			(xy 339.09 63.5) (xy 344.17 63.5)
 		)
@@
 	(wire
 		(pts
+			(xy 201.93 68.58) (xy 204.47 68.58)
+		)
+		(stroke
+			(width 0)
+			(type default)
+		)
+	)
+	(wire
+		(pts
 			(xy 403.86 43.18) (xy 403.86 41.91)
 		)
@@
 	(wire
 		(pts
+			(xy 201.93 68.58) (xy 200.66 68.58)
+		)
+		(stroke
+			(width 0)
+			(type default)
+		)
+	)
+	(wire
+		(pts
 			(xy 72.39 175.26) (xy 100.33 175.26)
 		)
@@
 	(global_label "P0.04"
 		(shape input)
-		(at 200.66 68.58 0)
+		(at 204.47 68.58 0)
 		(fields_autoplaced yes)
 		(effects
@@
 		)
 		(property "Intersheetrefs" "${INTERSHEET_REFS}"
-			(at 209.1485 68.58 0)
+			(at 212.9585 68.58 0)
 			(effects
 				(font
@@
 		(on_board yes)
 		(dnp no)
-		(property "Reference" "P1.9"
+		(property "Reference" "P1.09"
 			(at 57.658 220.726 90)
 			(effects
@@
 			(project "ESC_Texas"
 				(path "/0e3a5351-d2cd-4ecc-a1be-cca9c5f62ea0"
-					(reference "P1.9")
+					(reference "P1.09")
 					(unit 1)
 				)
@@
 	)
 	(symbol
+		(lib_id "Device:R")
+		(at 196.85 68.58 270)
+		(mirror x)
+		(unit 1)
+		(exclude_from_sim no)
+		(in_bom yes)
+		(on_board yes)
+		(dnp no)
+		(property "Reference" "R31"
+			(at 195.072 64.008 90)
+			(effects
+				(font
+					(size 1.27 1.27)
+				)
+				(justify left)
+			)
+		)
+		(property "Value" "R"
+			(at 196.088 66.294 90)
+			(effects
+				(font
+					(size 1.27 1.27)
+				)
+				(justify left)
+			)
+		)
+		(property "Footprint" "Resistor_SMD:R_0805_2012Metric"
+			(at 196.85 70.358 90)
+			(effects
+				(font
+					(size 1.27 1.27)
+				)
+				(hide yes)
+			)
+		)
+		(property "Datasheet" "~"
+			(at 196.85 68.58 0)
+			(effects
+				(font
+					(size 1.27 1.27)
+				)
+				(hide yes)
+			)
+		)
+		(property "Description" ""
+			(at 196.85 68.58 0)
+			(effects
+				(font
+					(size 1.27 1.27)
+				)
+				(hide yes)
+			)
+		)
+		(pin "1"
+		)
+		(pin "2"
+		)
+		(instances
+			(project "ESC_Texas"
+				(path "/0e3a5351-d2cd-4ecc-a1be-cca9c5f62ea0"
+					(reference "R31")
+					(unit 1)
+				)
+			)
+		)
+	)
+	(symbol
 		(lib_id "Connector:Conn_01x01_Pin")
 		(at 81.28 243.84 0)
@@
 	)
 	(symbol
+		(lib_id "Device:C")
+		(at 201.93 74.93 0)
+		(unit 1)
+		(exclude_from_sim no)
+		(in_bom yes)
+		(on_board yes)
+		(dnp no)
+		(property "Reference" "C19"
+			(at 207.264 74.93 0)
+			(effects
+				(font
+					(size 1.27 1.27)
+				)
+			)
+		)
+		(property "Value" "F"
+			(at 207.264 76.962 0)
+			(effects
+				(font
+					(size 1.27 1.27)
+				)
+			)
+		)
+		(property "Footprint" "Capacitor_SMD:C_0805_2012Metric"
+			(at 202.8952 78.74 0)
+			(effects
+				(font
+					(size 1.27 1.27)
+				)
+				(hide yes)
+			)
+		)
+		(property "Datasheet" "~"
+			(at 201.93 74.93 0)
+			(effects
+				(font
+					(size 1.27 1.27)
+				)
+				(hide yes)
+			)
+		)
+		(property "Description" ""
+			(at 201.93 74.93 0)
+			(effects
+				(font
+					(size 1.27 1.27)
+				)
+				(hide yes)
+			)
+		)
+		(pin "1"
+		)
+		(pin "2"
+		)
+		(instances
+			(project "ESC_Texas"
+				(path "/0e3a5351-d2cd-4ecc-a1be-cca9c5f62ea0"
+					(reference "C19")
+					(unit 1)
+				)
+			)
+		)
+	)
+	(symbol
 		(lib_id "Device:R")
 		(at 242.57 351.79 0)
@@
 	)
 	(symbol
+		(lib_id "power:GND")
+		(at 201.93 78.74 0)
+		(mirror y)
+		(unit 1)
+		(exclude_from_sim no)
+		(in_bom yes)
+		(on_board yes)
+		(dnp no)
+		(property "Reference" "#PWR038"
+			(at 201.93 85.09 0)
+			(effects
+				(font
+					(size 1.27 1.27)
+				)
+				(hide yes)
+			)
+		)
+		(property "Value" "GND"
+			(at 201.93 82.804 0)
+			(effects
+				(font
+					(size 1.27 1.27)
+				)
+			)
+		)
+		(property "Footprint" ""
+			(at 201.93 78.74 0)
+			(effects
+				(font
+					(size 1.27 1.27)
+				)
+				(hide yes)
+			)
+		)
+		(property "Datasheet" ""
+			(at 201.93 78.74 0)
+			(effects
+				(font
+					(size 1.27 1.27)
+				)
+				(hide yes)
+			)
+		)
+		(property "Description" "Power symbol creates a global label with name \"GND\" , ground"
+			(at 201.93 78.74 0)
+			(effects
+				(font
+					(size 1.27 1.27)
+				)
+				(hide yes)
+			)
+		)
+		(pin "1"
+		)
+		(instances
+			(project "ESC_Texas"
+				(path "/0e3a5351-d2cd-4ecc-a1be-cca9c5f62ea0"
+					(reference "#PWR038")
+					(unit 1)
+				)
+			)
+		)
+	)
+	(symbol
 		(lib_id "Device:LED")
 		(at 455.93 68.58 0)
@@
 		(on_board yes)
 		(dnp no)
-		(property "Reference" "P0.7"
+		(property "Reference" "P0.07"
 			(at 57.658 225.806 90)
 			(effects
@@
 			(project "ESC_Texas"
 				(path "/0e3a5351-d2cd-4ecc-a1be-cca9c5f62ea0"
-					(reference "P0.7")
+					(reference "P0.07")
 					(unit 1)
 				)

Commit message: Added reset button
Parts:
- removed JP3, JP4: SolderJumper_2_Open, Jumper:SolderJumper-2_P1.3mm_Open_Pad1.0x1.5mm, symbol Jumper:SolderJumper_2_Open
- added C52: F, Capacitor_SMD:C_0805_2012Metric, symbol Device:C
- added R32: 10k, Resistor_SMD:R_0805_2012Metric, symbol Device:R
- added SW1: 222AMVBAR, 222AMVBAR:SO4_222A-M-V-B_CTS, symbol 2024-11-13_14-35-25:222AMVBAR
- X2: footprint XRCGB32M000F2P29R0:XRCGB -> Package_SO:VSO-40_7.6x15.4mm_P0.762mm
Connections:
- net +10V: now also C52.1
- net +5V: now also U2.3 (VDD); no longer IC16.1 (VOUT)
- net GND: now also C52.2, SW1.3, SW1.4
- net VDD: now also R32.2
- net VDD_can: no longer U2.3 (VDD)
- net nRESET: now also R32.1, SW1.1, SW1.2
- new net +5V-c: IC16.1 (VOUT)
Other:
- note removed: "Digital I/O General purpose I/O"
- note removed: "General purpose I/O Analog input"
- note removed: "General purpose I/O Analog input Standard drive, low frequency I/O only"
- moved on the sheet: C38, C40, C41, D13, D14, H1, H2, H3, H4, IC12, J11, J2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
