File: ESC_Texas/Driver_subsheet.kicad_sch (KiCad schematic)
At the start: 24 parts, among them IC10 UCC21331CQDRQ1, Q5 IPD100N06S4, Q6 IPD100N06S4

Commit message: Done
Parts:
- added D17: RBR10BGE60ATL, RBR10BGE60ATL:RD3P175SNFRATL, symbol RBR10BGE60ATL:RBR10BGE60ATL
Connections:
- net +36V: now also D17.2 (K)
- net SW: now also D17.1 (A_1), D17.3 (A_2)
Other:
- moved on the sheet: C_3IN3
